Commit message: servo dummy publishes to rviz model

File: src/robot_arm/urdf/robot_arm.urdf (robot description, URDF)
Before this commit: robot visual, 4 links, 3 joints
Joints:
- joint link1_to_link2: axis 0 1 0 -> 0 -1 0

Commit message: mark drawings in orange

File: src/robot_arm/urdf/robot_arm.urdf (robot description, URDF)
Before this commit: robot visual, 4 links, 3 joints
Joints:
- joint base_to_link1: origin xyz=0.1011 -0.1236 0.37 -> xyz=0 0 0
